File: differential_bfp650_amp_hierarchy/simp_test/simp_test.sch (KiCad schematic (older format))
At the start: 9 parts

Commit message: Tuned simulation. Added extra RC in collector of differential amplifier output buffer. Tuned values to restore stability
Simulating 10 SiPM in parallel by increasing number of pixels x10 w.r.t.
model of single 3x3mm^2 SiPM

Peaking time ~ 800ns
Gain ~ 1 mV per Pixel Avalanche.
Parts:
- removed C1, C2: 100n, symbol Device:C
- removed R1: 100k, symbol Device:R
- removed R3, R4: 100, symbol Device:R
- D1: symbol d_sipm:D_SiPM -> simp_test-rescue:D_SiPM-d_sipm
- R2: value 100k -> 50
Connections:
- net vk: now also V1.1 (E1)
Changed lines of the file:
@@
 +PSPICE\n.control\noption savecurrents\ntran 1ns 500ns\nwrite\n.endc
 $Comp
-L d_sipm:D_SiPM D1
+L simp_test-rescue:D_SiPM-d_sipm D1
 U 1 1 5C338FC0
 P 5550 3200
@@
 	0    -1   1    0
 $EndComp
-Wire Wire Line
-	5550 3000 5550 2850
-Wire Wire Line
-	5550 3300 5550 3450
 $Comp
 L pspice:0 #GND02
@@
 	4800 3150 5300 3150
 $Comp
-L Device:R R1
-U 1 1 5C34507A
-P 5550 2600
-F 0 "R1" H 5480 2554 50  0000 R CNN
-F 1 "100k" H 5480 2645 50  0000 R CNN
-F 2 "" V 5480 2600 50  0001 C CNN
-F 3 "~" H 5550 2600 50  0001 C CNN
-	1    5550 2600
-	-1   0    0    1
-$EndComp
-$Comp
 L Device:R R2
 U 1 1 5C3451DD
 P 5550 3700
 F 0 "R2" H 5620 3746 50  0000 L CNN
-F 1 "100k" H 5620 3655 50  0000 L CNN
+F 1 "50" H 5620 3655 50  0000 L CNN
 F 2 "" V 5480 3700 50  0001 C CNN
 F 3 "~" H 5550 3700 50  0001 C CNN
@@
 Wire Wire Line
 	5550 3950 5550 3850
-Wire Wire Line
-	5550 3550 5550 3450
-Connection ~ 5550 3450
-Wire Wire Line
-	5550 2850 5550 2750
-Connection ~ 5550 2850
-Wire Wire Line
-	5550 2450 5550 2300
 Wire Wire Line
 	5550 2300 4250 2300
@@
 Text Label 5550 3350 0    50   ~ 0
 va
-$Comp
-L Device:R R3
-U 1 1 5C350FD5
-P 6350 2850
-F 0 "R3" V 6143 2850 50  0000 C CNN
-F 1 "100" V 6234 2850 50  0000 C CNN
-F 2 "" V 6280 2850 50  0001 C CNN
-F 3 "~" H 6350 2850 50  0001 C CNN
-	1    6350 2850
-	0    1    1    0
-$EndComp
 Wire Wire Line
-	5550 2850 5750 2850
+	5550 2300 5550 3000
 Wire Wire Line
-	5550 3450 5750 3450
-$Comp
-L Device:C C1
-U 1 1 5C351382
-P 5900 2850
-F 0 "C1" V 5648 2850 50  0000 C CNN
-F 1 "100n" V 5739 2850 50  0000 C CNN
-F 2 "" H 5938 2700 50  0001 C CNN
-F 3 "~" H 5900 2850 50  0001 C CNN
-	1    5900 2850
-	0    1    1    0
-$EndComp
-Wire Wire Line
-	6050 2850 6200 2850
-$Comp
-L Device:C C2
-U 1 1 5C351457
-P 5900 3450
-F 0 "C2" V 5648 3450 50  0000 C CNN
-F 1 "100n" V 5739 3450 50  0000 C CNN
-F 2 "" H 5938 3300 50  0001 C CNN
-F 3 "~" H 5900 3450 50  0001 C CNN
-	1    5900 3450
-	0    1    1    0
-$EndComp
-Wire Wire Line
-	6050 3450 6200 3450
-$Comp
-L Device:R R4
-U 1 1 5C351928
-P 6350 3450
-F 0 "R4" V 6143 3450 50  0000 C CNN
-F 1 "100" V 6234 3450 50  0000 C CNN
-F 2 "" V 6280 3450 50  0001 C CNN
-F 3 "~" H 6350 3450 50  0001 C CNN
-	1    6350 3450
-	0    1    1    0
-$EndComp
-$Comp
-L pspice:0 #GND0101
-U 1 1 5C3519A3
-P 6650 3250
-F 0 "#GND0101" H 6650 3150 50  0001 C CNN
-F 1 "0" H 6650 3337 50  0000 C CNN
-F 2 "" H 6650 3250 50  0001 C CNN
-F 3 "~" H 6650 3250 50  0001 C CNN
-	1    6650 3250
-	1    0    0    -1
-$EndComp
-Wire Wire Line
-	6500 2850 6550 2850
-Wire Wire Line
-	6550 2850 6550 3100
-Wire Wire Line
-	6550 3450 6500 3450
-Wire Wire Line
-	6650 3250 6650 3100
-Wire Wire Line
-	6650 3100 6550 3100
-Connection ~ 6550 3100
-Wire Wire Line
-	6550 3100 6550 3450
+	5550 3300 5550 3550
 $EndSCHEMATC
